File: Eagle Files/SunriseClockSwitchesv2.brd (EAGLE design)
At the start: 55.4 x 16.8 mm, 7 parts

Commit message: Adding drawings
Parts:
- moved FROMSWITCHES 29.2 mm to (25.0, 1.91)
- moved SWITCH 10.2 mm to (15.2, 8.00)
Routing:
- net STOP: track 55.1 -> 11.7 mm
- net VCC: track 48.6 -> 9.18 mm
- net ROT_B: track 39.5 -> 20.8 mm
- net GND: track 48.8 -> 34.0 mm
- net ROTSW: track 15.1 -> 28.5 mm, vias 1 -> 0
- net N$13: track 26.7 -> 18.8 mm
- net ROT_A: track 37.1 -> 36.2 mm
Other:
- board size 55.4 x 16.8 mm -> 42.7 x 16.8 mm
