File: Eagle Files/SunriseClockMainv3.brd (EAGLE design)
At the start: 33.1 x 30.1 mm, 8 parts

Commit message: Updated eagle files and schematic
Parts:
- added DC1: BP5293-50, dc-dc-converter:SIP3
- added N-MOS1: (no value), SparkFun-DiscreteSemi:TO220V
- added R2: 100, SparkFun-Resistors:AXIAL-0.4
- added R3, R4: 100K, SparkFun-Resistors:AXIAL-0.4
- R1: value 2.2K -> 100
- moved R1 8.89 mm to (6.99, 48.3)
- moved RTC 7.67 mm to (21.6, 66.0)
- moved TO_SW 5.08 mm to (18.4, 62.9)
- moved 3208 4.62 mm to (18.4, 59.1)
- moved N-MOS 0.63 mm to (12.7, 59.1)
Connections:
- removed net VCC: 3208.2, PRO_MICRO.21, RTC.2, TO_SW.2
- new net 5V: 3208.2, DC1.3, RTC.2, TO_SW.2
- new net N$2: N-MOS1.1, R2.P$2, R3.P$2
- new net POWERFET: N-MOS1.3, R1.P$1
- net GND: now also DC1.2, R3.P$1, R4.P$1
- net LEDSIG: now also R2.P$1; no longer R1.P$1
- net N$1: now also R4.P$2
- net RAW: now also DC1.1, N-MOS1.2
Routing:
- net N$2: track 0.00 -> 31.4 mm
- net GND: track 46.9 -> 76.4 mm
- net POWERFET: track 0.00 -> 23.5 mm
- net VCC: track 21.2 -> 0.00 mm
- net SCL: track 22.2 -> 37.1 mm
- net 5V: track 0.00 -> 13.8 mm
- net N$1: track 18.1 -> 30.8 mm
- net SDA: track 22.5 -> 34.8 mm, vias 0 -> 1
- net RAW: track 17.7 -> 28.3 mm
- net ROT_B: track 18.9 -> 13.2 mm
- net ROT_A: track 12.6 -> 7.52 mm
- net LEDSIG: track 39.4 -> 34.7 mm
- net STOP: track 28.9 -> 24.3 mm
- net SQW: track 52.2 -> 56.5 mm
- net WR: track 10.2 -> 8.23 mm
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Other:
- board text added: "1"
- board text added: "In"
