File: Eagle Files/SunriseClockMainv3.sch (EAGLE design)
At the start: 8 parts

Commit message: Updated eagle files and schematic
Parts:
- added DC1: BP5293-50, dc-dc-converter:R-78C5.0-1.0
- added N-MOS1: MOSFET-NCHANNELFQP30N06L, SparkFun-DiscreteSemi:MOSFET-NCHANNELFQP30N06L
- added R2: 100, SparkFun-Resistors:RESISTORPTH-1/4W
- added R3, R4: 100K, SparkFun-Resistors:RESISTORPTH-1/4W
- R1: value 2.2K -> 100
Connections:
- removed net VCC: 3208.2, PRO_MICRO.VCC, RTC.2, TO_SW.2
- new net 5V: 3208.2, DC1.VOUT, RTC.2, TO_SW.2
- new net N$2: N-MOS1.G, R2.2, R3.2
- new net POWERFET: N-MOS1.S, R1.1
- net GND: now also DC1.GND, R3.1, R4.1
- net LEDSIG: now also R2.1; no longer R1.1
- net N$1: now also R4.2
- net RAW: now also DC1.VIN, N-MOS1.D
Other:
- moved on the sheet: N-MOS, R1
